File: cat-tracker-board.sch (KiCad schematic (older format))
At the start: 1 part

Commit message: Added MCU and friends and connected to radio.
Parts:
- added C?: 1 uF, symbol Device:C
- added C? (x3): 0.1 uF, symbol Device:C
- added C? (x2): 15 pF, symbol Device:C
- added FB?: Ferrite_Bead, symbol Device:Ferrite_Bead
- added J?: Conn_01x10, symbol Connector_Generic:Conn_01x10
- added R? (x2): 2.2 K, symbol Device:R
- added U?: ATSAMD21G18A-AUT, Package_QFP:TQFP-48_7x7mm_P0.5mm, symbol MCU_Microchip_SAMD:ATSAMD21G18A-AUT
- added Y?: 32.768 kHz, symbol Device:Crystal
Connections:
- net labels added: +3V3, GND, MISO, MOSI, NSS, RFM_INT, RFM_RESET, SCK, SWCLK, SWDIO, nRESET
- wire segments 0 -> 62
Other:
- moved on the sheet: U?

Commit message: Changed mcu to 32 pin, added usb, power.
Parts:
- removed C?: 0.1 uF, symbol Device:C
- removed C? (x2): 15 pF, symbol Device:C
- removed U?: ATSAMD21G18A-AUT, Package_QFP:TQFP-48_7x7mm_P0.5mm, symbol MCU_Microchip_SAMD:ATSAMD21G18A-AUT
- removed Y?: 32.768 kHz, symbol Device:Crystal
- added BT?: Battery, symbol Device:Battery
- added C? (x2): 10 uF, symbol Device:C
- added C? (x2): 0.1 uF, symbol Device:C
- added C? (x2): 4.7 uF, symbol Device:C
- added J?: USB_C_Receptacle_USB2.0, symbol Connector:USB_C_Receptacle_USB2.0
- added L?: 4.7 uH, symbol Device:L
- added Q?: Q_PMOS_GSD, Package_TO_SOT_SMD:SOT-23, symbol Device:Q_PMOS_GSD
- added R? (x2): 5.1 K, symbol Device:R
- added R?: 2.2 K, symbol Device:R
- added U?: ATSAMD21E18A-A, Package_QFP:TQFP-32_7x7mm_P0.8mm, symbol MCU_Microchip_SAMD:ATSAMD21E18A-A
- added U?: LM3480-3.3, Package_TO_SOT_SMD:SOT-23, symbol Regulator_Linear:LM3480-3.3
- added U?: AAT1217IGU-3.3, Package_TO_SOT_SMD:SOT-23-6, symbol Regulator_Switching:AAT1217IGU-3.3
Connections:
- net labels added: +5V, USBDM, USBDP, VBAT, VBAT_SW, VUSB
- wire segments 62 -> 96
Other:
- moved on the sheet: C?, FB?, J?, R?, U?

Commit message: Added some part numbers, updated boost regulator to a part that's not obsolete.
Parts:
- removed U?: AAT1217IGU-3.3, Package_TO_SOT_SMD:SOT-23-6, symbol Regulator_Switching:AAT1217IGU-3.3
- added U?: TPS61097A-33DBVR, Package_TO_SOT_SMD:SOT-23-5, symbol colinholzman:TPS61097A-33DBVR
- C? (x2): value 4.7 uF -> 10 uF
- J?: footprint (none) -> Connector_USB:USB_C_Receptacle_Amphenol_12401610E4-2A; mfg1 (none) -> Amphenol; mfg1pn (none) -> 12401610E4#2A
- U?: mfg1 (none) -> RF Solutions; mfg1pn (none) -> RFM95W-915S2
- U?: mfg1 (none) -> Texas Instruments; mfg1pn (none) -> LM3480IM3-3.3/NOPB
Connections:
- wire segments 96 -> 97
Other:
- moved on the sheet: C?, L?
Changed lines of the file:
@@
 F 2 "" H 11400 6200 50  0001 C CNN
 F 3 "https://www.hoperf.com/data/upload/portal/20181127/5bfcbea20e9ef.pdf" H 11400 6200 50  0001 C CNN
+F 4 "RF Solutions" H 14700 4550 50  0001 C CNN "mfg1"
+F 5 "RFM95W-915S2" H 14700 4550 50  0001 C CNN "mfg1pn"
 	1    14700 4550
 	1    0    0    -1
@@
 F 0 "J?" H 14320 1689 50  0000 R CNN
 F 1 "USB_C_Receptacle_USB2.0" H 14320 1598 50  0000 R CNN
-F 2 "" H 14900 1750 50  0001 C CNN
+F 2 "Connector_USB:USB_C_Receptacle_Amphenol_12401610E4-2A" H 14900 1750 50  0001 C CNN
 F 3 "https://www.usb.org/sites/default/files/documents/usb_type-c.zip" H 14900 1750 50  0001 C CNN
+F 4 "Amphenol" H 14750 1750 50  0001 C CNN "mfg1"
+F 5 "12401610E4#2A" H 14750 1750 50  0001 C CNN "mfg1pn"
 	1    14750 1750
 	-1   0    0    -1
@@
 F 2 "Package_TO_SOT_SMD:SOT-23" H 9950 1825 50  0001 C CIN
 F 3 "http://www.ti.com/lit/ds/symlink/lm3480.pdf" H 9950 1600 50  0001 C CNN
+F 4 "Texas Instruments" H 9950 1600 50  0001 C CNN "mfg1"
+F 5 "LM3480IM3-3.3/NOPB" H 9950 1600 50  0001 C CNN "mfg1pn"
 	1    9950 1600
 	1    0    0    -1
@@
 Text HLabel 8650 3550 0    50   Input ~ 0
 VUSB
-$Comp
-L Regulator_Switching:AAT1217IGU-3.3 U?
-U 1 1 6096F1A4
-P 10700 3400
-F 0 "U?" H 10450 3650 50  0000 C CNN
-F 1 "AAT1217IGU-3.3" H 11100 3650 50  0000 C CNN
-F 2 "Package_TO_SOT_SMD:SOT-23-6" H 10700 3400 50  0001 C CNN
-F 3 "http://www.skyworksinc.com/uploads/documents/AAT1217_202050B.pdf" H 10700 3400 50  0001 C CNN
-F 4 "Skyworks" H 10700 3400 50  0001 C CNN "mfg1"
-F 5 "AAT1217IGU-3.3-T1 " H 10700 3400 50  0001 C CNN "mfg1pn"
-	1    10700 3400
-	1    0    0    -1
-$EndComp
 Wire Wire Line
 	8900 3200 8950 3200
 Text HLabel 8950 3200 2    50   Input ~ 0
 VBAT_SW
-Wire Wire Line
-	10300 3300 10250 3300
-Text HLabel 10200 3300 0    50   Input ~ 0
+Text HLabel 10100 3200 0    50   Input ~ 0
 VBAT_SW
 Wire Wire Line
-	10300 3500 10250 3500
-Wire Wire Line
-	10250 3500 10250 3300
-Connection ~ 10250 3300
-Wire Wire Line
-	10250 3300 10200 3300
-Wire Wire Line
-	11100 3300 11250 3300
-Text HLabel 11300 3300 2    50   Input ~ 0
-+3V3
-Wire Wire Line
-	10250 3850 10250 3900
-Text HLabel 10250 3900 3    50   Input ~ 0
+	11350 3300 11400 3300
+Text HLabel 11450 3300 2    50   Input ~ 0
++3V3
+Wire Wire Line
+	10150 4050 10150 4100
+Text HLabel 10150 4100 3    50   Input ~ 0
 GND
 $Comp
 L Device:C C?
 U 1 1 609853E4
-P 10250 3700
-F 0 "C?" V 9998 3700 50  0000 C CNN
-F 1 "4.7 uF" V 10089 3700 50  0000 C CNN
-F 2 "" H 10288 3550 50  0001 C CNN
-F 3 "~" H 10250 3700 50  0001 C CNN
-	1    10250 3700
+P 10150 3900
+F 0 "C?" V 9898 3900 50  0000 C CNN
+F 1 "10 uF" V 9989 3900 50  0000 C CNN
+F 2 "" H 10188 3750 50  0001 C CNN
+F 3 "~" H 10150 3900 50  0001 C CNN
+	1    10150 3900
 	1    0    0    1
 $EndComp
-Wire Wire Line
-	10250 3550 10250 3500
-Connection ~ 10250 3500
 $Comp
 L Device:L L?
 U 1 1 60989E09
-P 10450 3000
-F 0 "L?" V 10269 3000 50  0000 C CNN
-F 1 "4.7 uH" V 10360 3000 50  0000 C CNN
-F 2 "" H 10450 3000 50  0001 C CNN
-F 3 "~" H 10450 3000 50  0001 C CNN
-	1    10450 3000
+P 10350 3500
+F 0 "L?" V 10150 3500 50  0000 C CNN
+F 1 "4.7 uH" V 10250 3500 50  0000 C CNN
+F 2 "" H 10350 3500 50  0001 C CNN
+F 3 "~" H 10350 3500 50  0001 C CNN
+	1    10350 3500
 	0    1    1    0
 $EndComp
 Wire Wire Line
-	10700 3700 10700 3750
-Text HLabel 10700 3750 3    50   Input ~ 0
-GND
-Wire Wire Line
-	10600 3000 10700 3000
-Wire Wire Line
-	10700 3000 10700 3100
-Wire Wire Line
-	10300 3000 10250 3000
-Wire Wire Line
-	10250 3000 10250 3300
-Wire Wire Line
-	11250 3650 11250 3700
-Text HLabel 11250 3700 3    50   Input ~ 0
+	10950 3900 10950 3950
+Text HLabel 10950 3950 3    50   Input ~ 0
+GND
+Wire Wire Line
+	11400 3650 11400 3700
+Text HLabel 11400 3700 3    50   Input ~ 0
 GND
 $Comp
 L Device:C C?
 U 1 1 60994D70
-P 11250 3500
-F 0 "C?" H 11365 3454 50  0000 L CNN
-F 1 "4.7 uF" H 11365 3545 50  0000 L CNN
-F 2 "" H 11288 3350 50  0001 C CNN
-F 3 "~" H 11250 3500 50  0001 C CNN
-	1    11250 3500
+P 11400 3500
+F 0 "C?" H 11515 3454 50  0000 L CNN
+F 1 "10 uF" H 11515 3545 50  0000 L CNN
+F 2 "" H 11438 3350 50  0001 C CNN
+F 3 "~" H 11400 3500 50  0001 C CNN
+	1    11400 3500
 	1    0    0    1
 $EndComp
 Wire Wire Line
-	11250 3350 11250 3300
-Connection ~ 11250 3300
-Wire Wire Line
-	11250 3300 11300 3300
+	11400 3350 11400 3300
+Wire Wire Line
+	10100 3200 10150 3200
+Wire Wire Line
+	10500 3500 10550 3500
+Wire Wire Line
+	10200 3500 10150 3500
+Wire Wire Line
+	10150 3500 10150 3200
+Connection ~ 10150 3200
+Wire Wire Line
+	10150 3200 10500 3200
+Wire Wire Line
+	10150 3500 10150 3700
+Wire Wire Line
+	10150 3700 10550 3700
+Connection ~ 10150 3500
+Wire Wire Line
+	10150 3750 10150 3700
+Connection ~ 10150 3700
+Connection ~ 11400 3300
+Wire Wire Line
+	11400 3300 11450 3300
+Wire Wire Line
+	10500 3200 10500 3300
+Wire Wire Line
+	10500 3300 10550 3300
+$Comp
+L colinholzman:TPS61097A-33DBVR U?
+U 1 1 609EC946
+P 10950 3400
+F 0 "U?" H 10950 3767 50  0000 C CNN
+F 1 "TPS61097A-33DBVR" H 10950 3676 50  0000 C CNN
+F 2 "Package_TO_SOT_SMD:SOT-23-5" H 10950 2500 50  0001 C CNN
+F 3 "" H 10950 3250 50  0001 C CNN
+F 4 "Texas Instruments" H 10950 3400 50  0001 C CNN "mfg1"
+F 5 "TPS61097A-33DBVR" H 10950 3400 50  0001 C CNN "mfg1pn"
+	1    10950 3400
+	1    0    0    -1
+$EndComp
 $EndSCHEMATC

Commit message: Added low voltage cutoff circuit for batteries.
Parts:
- added C?: 0.1 uF, symbol Device:C
- added D? (x2): D, symbol Device:D
- added D?: D_Schottky, symbol Device:D_Schottky
- added Q?: SI3443DDV-T1-GE3, Package_SO:TSOP-6_1.65x3.05mm_P0.95mm, symbol colinholzman:Si3443
- added Q?: Q_NPN_BCE, symbol Device:Q_NPN_BCE
- added Q?: Q_PNP_BCE, symbol Device:Q_PNP_BCE
- added R? (x2): 500K, symbol Device:R
- added R?: 270K, symbol Device:R
- added R?: 100K, symbol Device:R
- Q?: value Q_PMOS_GSD -> SI3443DDV-T1-GE3; footprint Package_TO_SOT_SMD:SOT-23 -> Package_SO:TSOP-6_1.65x3.05mm_P0.95mm; symbol Device:Q_PMOS_GSD -> colinholzman:Si3443; mfg1 Nexperia -> Vishay Semiconductors; mfg1pn BSH202,215 -> SI3443DDV-T1-GE3
Connections:
- net +5V is gone; now on net VUSB: C?.2, J?.A4 (VBUS), J?.A9 (VBUS), J?.B4 (VBUS), J?.B9 (VBUS), U?.2 (VI)
- net +3V3: now also D?.2 (A)
- net GND: now also Q?.3 (E), R?.2
- net VBAT: now also Q?.4 (S); no longer Q?.2 (S)
- net VBAT_SW: now also Q?.1 (D), Q?.2 (D), Q?.5 (D), Q?.6 (D), C?.2, D?.2 (A), Q?.4 (S), R?.1, R?.1; no longer C?.2, L?.2, Q?.3 (D), U?.1 (VIN), U?.3 (EN)
- net VUSB: now also Q?.3 (G), D?.1 (K); no longer Q?.1 (G)
- new net: Q?.1 (B), Q?.2 (C), Q?.3 (G), R?.2
- new net: Q?.3 (E), R?.2
- new net: C?.1, D?.1 (K), R?.1
- new net: Q?.1 (B), Q?.2 (C), R?.1, R?.2
- new net: D?.1 (K), D?.2 (A)
- new net VBAT_LVP: C?.2, L?.2, Q?.1 (D), Q?.2 (D), Q?.5 (D), Q?.6 (D), U?.1 (VIN), U?.3 (EN)
Other:
- moved on the sheet: BT?, C?, L?, Q?, R?, U?

Commit message: Added GPS connector and switch, annotated symbols, and assigned footprints.
Parts:
- added J3: Conn_01x03, Connector_JST:JST_PH_S3B-PH-K_1x03_P2.00mm_Horizontal, symbol Connector_Generic:Conn_01x03
- added Q5: SI3443DDV-T1-GE3, Package_SO:TSOP-6_1.65x3.05mm_P0.95mm, symbol colinholzman:Si3443
- added R8: 100k, Resistor_SMD:R_0805_2012Metric, symbol Device:R
- BT1: renamed from BT?; footprint (none) -> Battery:BatteryHolder_Keystone_2468_2xAAA
- C1, C3, C5, C6, C7, C8: renamed from C?; footprint (none) -> Capacitor_SMD:C_0805_2012Metric
- C10, C2, C4, C9: renamed from C?; footprint (none) -> Capacitor_SMD:C_1210_3225Metric; mfg1 (none) -> Taiyo Yuden; mfg1pn (none) -> UMK325AB7106MMHP
- D1, D2: renamed from D?; footprint (none) -> Diode_SMD:D_SOD-123
- D3: renamed from D?; footprint (none) -> Diode_SMD:D_SOD-123; mfg1 (none) -> Vishay Semiconductors; mfg1pn (none) -> BAT54W-HG3-08
- FB1: renamed from FB?; footprint (none) -> Inductor_SMD:L_0805_2012Metric
- J1: renamed from J?; footprint (none) -> Connector_PinHeader_1.27mm:PinHeader_2x05_P1.27mm_Vertical
- L1: renamed from L?; footprint (none) -> Inductor_SMD:L_1008_2520Metric; mfg1 (none) -> Taiyo Yuden; mfg1pn (none) -> LBC2518T4R7M
- Q2, Q3: renamed from Q?; footprint (none) -> Package_TO_SOT_SMD:SOT-23
- R1, R2, R3: renamed from R?; value 2.2 K -> 100k; footprint (none) -> Resistor_SMD:R_0805_2012Metric
- R10, R9: renamed from R?; value 5.1 K -> 5.1k; footprint (none) -> Resistor_SMD:R_0805_2012Metric
- R4: renamed from R?; value 270K -> 270k; footprint (none) -> Resistor_SMD:R_0805_2012Metric
- R5: renamed from R?; value 100K -> 100k; footprint (none) -> Resistor_SMD:R_0805_2012Metric
- R6, R7: renamed from R?; value 500K -> 500k; footprint (none) -> Resistor_SMD:R_0805_2012Metric
- U4: renamed from U?; footprint (none) -> RF_Module:HOPERF_RFM9XW_SMD
- gave numbers to parts that had none: 6
Connections:
- net +3V3: now also Q5.4 (S), R8.2
- net GND: now also J3.2 (Pin_2)
- net GPS_TX: now reaches U1.17 (PA16)
- net GPS_TX: now also J3.1 (Pin_1)
- net GPS_EN: now reaches U1.18 (PA17)
- net GPS_EN: now also Q5.3 (G), R8.1
- new net GPS_PWR: J3.3 (Pin_3), Q5.1 (D), Q5.2 (D), Q5.5 (D), Q5.6 (D)

Commit message: Fixed BJT pin numbers.
Parts:
- Q2: symbol Device:Q_PNP_BCE -> Device:Q_PNP_BEC
- Q3: symbol Device:Q_NPN_BCE -> Device:Q_NPN_BEC
Connections:
- net GND: now also Q3.2 (E); no longer Q3.3 (E)
- net at Q2.1 (B), Q4.3 (G), R7.2: now also Q3.3 (C); no longer Q3.2 (C)
- net at R6.2: now also Q2.2 (E); no longer Q2.3 (E)
- net at Q3.1 (B), R4.2, R5.1: now also Q2.3 (C); no longer Q2.2 (C)
Changed lines of the file:
@@
 $EndComp
 $Comp
-L Device:Q_NPN_BCE Q3
+L Device:Q_NPN_BEC Q3
 U 1 1 608E668F
 P 9250 5900
@@
 $EndComp
 $Comp
-L Device:Q_PNP_BCE Q2
+L Device:Q_PNP_BEC Q2
 U 1 1 608E6F56
 P 9100 5650
