File: cat-tracker-board.kicad_pcb (KiCad board)
At the start: 2 copper layers, 15.2 x 10.2 mm, 38 parts, among them J1 Conn_01x10, J2 USB_C_Receptacle_USB2.0, J3 Conn_01x03, Q1 SI3443DDV-T1-GE3, Q2 Q_PNP_BCE, Q3 Q_NPN_BCE, Q4 SI3443DDV-T1-GE3, Q5 SI3443DDV-T1-GE3, U1 ATSAMD21E18A-A, U2 LM3480-3.3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

Commit message: Updated pcb with new BJT nets.
Connections:
- Q3 pad 1: Net-(Q2-Pad2) -> Net-(Q2-Pad3)
- Q3 pad 2: Net-(Q2-Pad1) -> /GND
- Q3 pad 3: /GND -> Net-(Q2-Pad1)
- R4 pad 2: Net-(Q2-Pad2) -> Net-(Q2-Pad3)
- R5 pad 1: Net-(Q2-Pad2) -> Net-(Q2-Pad3)
- R6 pad 2: Net-(Q2-Pad3) -> Net-(Q2-Pad2)
Changed lines of the file:
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@@
     (fp_line (start 1.68 0.95) (end -1.68 0.95) (layer F.CrtYd) (width 0.05))
     (pad 2 smd roundrect (at 0.9125 0) (size 1.025 1.4) (layers F.Cu F.Paste F.Mask) (roundrect_rratio 0.243902)
+      (net 28 "Net-(Q2-Pad2)"))
+    (pad 1 smd roundrect (at -0.9125 0) (size 1.025 1.4) (layers F.Cu F.Paste F.Mask) (roundrect_rratio 0.243902)
+      (net 6 /VBAT_SW))
+    (model ${KISYS3DMOD}/Resistor_SMD.3dshapes/R_0805_2012Metric.wrl
+      (at (xyz 0 0 0))
+      (scale (xyz 1 1 1))
+      (rotate (xyz 0 0 0))
+    )
+  )
+  (module Resistor_SMD:R_0805_2012Metric (layer F.Cu)
+    (at 81.78 32.78)
+    (descr "Resistor SMD 0805 (2012 Metric), square (rectangular) end terminal, IPC_7351 nominal, (Body size source: IPC-SM-782 page 72, https://www.pcb-3d.com/wordpress/wp-content/uploads/ipc-sm-782a_amendment_1_and_2.pdf), generated with kicad-footprint-generator")
+    (tags resistor)
+    (attr smd)
+    (fp_text reference R5 (at 0 -1.65) (layer F.SilkS)
+      (effects (font (size 1 1) (thickness 0.15)))
+    )
+    (fp_text value 100k (at 0 1.65) (layer F.Fab)
+      (effects (font (size 1 1) (thickness 0.15)))
+    )
+    (fp_text user %R (at 0 0) (layer F.Fab)
+      (effects (font (size 0.5 0.5) (thickness 0.08)))
+    )
+    (fp_line (start -1 0.625) (end -1 -0.625) (layer F.Fab) (width 0.1))
+    (fp_line (start -1 -0.625) (end 1 -0.625) (layer F.Fab) (width 0.1))
+    (fp_line (start 1 -0.625) (end 1 0.625) (layer F.Fab) (width 0.1))
+    (fp_line (start 1 0.625) (end -1 0.625) (layer F.Fab) (width 0.1))
+    (fp_line (start -0.227064 -0.735) (end 0.227064 -0.735) (layer F.SilkS) (width 0.12))
+    (fp_line (start -0.227064 0.735) (end 0.227064 0.735) (layer F.SilkS) (width 0.12))
+    (fp_line (start -1.68 0.95) (end -1.68 -0.95) (layer F.CrtYd) (width 0.05))
+    (fp_line (start -1.68 -0.95) (end 1.68 -0.95) (layer F.CrtYd) (width 0.05))
+    (fp_line (start 1.68 -0.95) (end 1.68 0.95) (layer F.CrtYd) (width 0.05))
+    (fp_line (start 1.68 0.95) (end -1.68 0.95) (layer F.CrtYd) (width 0.05))
+    (pad 2 smd roundrect (at 0.9125 0) (size 1.025 1.4) (layers F.Cu F.Paste F.Mask) (roundrect_rratio 0.243902)
+      (net 1 /GND))
+    (pad 1 smd roundrect (at -0.9125 0) (size 1.025 1.4) (layers F.Cu F.Paste F.Mask) (roundrect_rratio 0.243902)
       (net 27 "Net-(Q2-Pad3)"))
-    (pad 1 smd roundrect (at -0.9125 0) (size 1.025 1.4) (layers F.Cu F.Paste F.Mask) (roundrect_rratio 0.243902)
-      (net 6 /VBAT_SW))
-    (model ${KISYS3DMOD}/Resistor_SMD.3dshapes/R_0805_2012Metric.wrl
-      (at (xyz 0 0 0))
-      (scale (xyz 1 1 1))
-      (rotate (xyz 0 0 0))
-    )
-  )
-  (module Resistor_SMD:R_0805_2012Metric (layer F.Cu)
-    (at 81.78 32.78)
-    (descr "Resistor SMD 0805 (2012 Metric), square (rectangular) end terminal, IPC_7351 nominal, (Body size source: IPC-SM-782 page 72, https://www.pcb-3d.com/wordpress/wp-content/uploads/ipc-sm-782a_amendment_1_and_2.pdf), generated with kicad-footprint-generator")
-    (tags resistor)
-    (attr smd)
-    (fp_text reference R5 (at 0 -1.65) (layer F.SilkS)
-      (effects (font (size 1 1) (thickness 0.15)))
-    )
-    (fp_text value 100k (at 0 1.65) (layer F.Fab)
-      (effects (font (size 1 1) (thickness 0.15)))
-    )
-    (fp_text user %R (at 0 0) (layer F.Fab)
-      (effects (font (size 0.5 0.5) (thickness 0.08)))
-    )
-    (fp_line (start -1 0.625) (end -1 -0.625) (layer F.Fab) (width 0.1))
-    (fp_line (start -1 -0.625) (end 1 -0.625) (layer F.Fab) (width 0.1))
-    (fp_line (start 1 -0.625) (end 1 0.625) (layer F.Fab) (width 0.1))
-    (fp_line (start 1 0.625) (end -1 0.625) (layer F.Fab) (width 0.1))
-    (fp_line (start -0.227064 -0.735) (end 0.227064 -0.735) (layer F.SilkS) (width 0.12))
-    (fp_line (start -0.227064 0.735) (end 0.227064 0.735) (layer F.SilkS) (width 0.12))
-    (fp_line (start -1.68 0.95) (end -1.68 -0.95) (layer F.CrtYd) (width 0.05))
-    (fp_line (start -1.68 -0.95) (end 1.68 -0.95) (layer F.CrtYd) (width 0.05))
-    (fp_line (start 1.68 -0.95) (end 1.68 0.95) (layer F.CrtYd) (width 0.05))
-    (fp_line (start 1.68 0.95) (end -1.68 0.95) (layer F.CrtYd) (width 0.05))
-    (pad 2 smd roundrect (at 0.9125 0) (size 1.025 1.4) (layers F.Cu F.Paste F.Mask) (roundrect_rratio 0.243902)
-      (net 1 /GND))
-    (pad 1 smd roundrect (at -0.9125 0) (size 1.025 1.4) (layers F.Cu F.Paste F.Mask) (roundrect_rratio 0.243902)
-      (net 28 "Net-(Q2-Pad2)"))
     (model ${KISYS3DMOD}/Resistor_SMD.3dshapes/R_0805_2012Metric.wrl
       (at (xyz 0 0 0))
@@
     (fp_line (start 1.68 0.95) (end -1.68 0.95) (layer F.CrtYd) (width 0.05))
     (pad 2 smd roundrect (at 0.9125 0) (size 1.025 1.4) (layers F.Cu F.Paste F.Mask) (roundrect_rratio 0.243902)
-      (net 28 "Net-(Q2-Pad2)"))
+      (net 27 "Net-(Q2-Pad3)"))
     (pad 1 smd roundrect (at -0.9125 0) (size 1.025 1.4) (layers F.Cu F.Paste F.Mask) (roundrect_rratio 0.243902)
       (net 7 "Net-(C6-Pad1)"))
@@
     (fp_line (start 0.76 1.58) (end -0.7 1.58) (layer F.SilkS) (width 0.12))
     (pad 3 smd rect (at 1 0) (size 0.9 0.8) (layers F.Cu F.Paste F.Mask)
+      (net 29 "Net-(Q2-Pad1)"))
+    (pad 2 smd rect (at -1 0.95) (size 0.9 0.8) (layers F.Cu F.Paste F.Mask)
       (net 1 /GND))
-    (pad 2 smd rect (at -1 0.95) (size 0.9 0.8) (layers F.Cu F.Paste F.Mask)
-      (net 29 "Net-(Q2-Pad1)"))
     (pad 1 smd rect (at -1 -0.95) (size 0.9 0.8) (layers F.Cu F.Paste F.Mask)
-      (net 28 "Net-(Q2-Pad2)"))
+      (net 27 "Net-(Q2-Pad3)"))
     (model ${KISYS3DMOD}/Package_TO_SOT_SMD.3dshapes/SOT-23.wrl
       (at (xyz 0 0 0))
