File: battery-board/battery-board.sch (KiCad schematic (older format))
At the start: 1 part

Commit message: Updated battery board pns and added aux bom.
Parts:
- BT1: mfg1 (none) -> Keystone; mfg1pn (none) -> 2468
Changed lines of the file:
@@
 F 2 "Battery:BatteryHolder_Keystone_2468_2xAAA" V 5750 3660 50  0001 C CNN
 F 3 "~" V 5750 3660 50  0001 C CNN
+F 4 "Keystone" H 5750 3600 50  0001 C CNN "mfg1"
+F 5 "2468" H 5750 3600 50  0001 C CNN "mfg1pn"
 	1    5750 3600
 	1    0    0    -1
