File: main-board/cat-tracker-board.sch (KiCad schematic (older format))
At the start: 28 parts, among them J1 Conn_01x10, J2 USB_C_Receptacle_USB2.0, J3 Conn_01x03, J4 Conn_01x02, Q5 SI3443DDV-T1-GE3, SW1 PCM12SMTR, U1 ATSAMD21E18A-A, U2 LM3480-3.3, U3 TPS61097A-33DBVR, U4 RFM95W-915S2

Commit message: Remove boost converter, replace with low Vf schottky.
Parts:
- removed C10, C9: 10 uF, Capacitor_SMD:C_1210_3225Metric, symbol Device:C
- removed L1: 10 uH, colinholzman:DO3314-...MLC, symbol Device:L
- removed U3: TPS61097A-33DBVR, Package_TO_SOT_SMD:SOT-23-5, symbol colinholzman:TPS61097A-33DBVR
- added D1: CUS08F30, Diode_SMD:D_SOD-323_HandSoldering, symbol Device:D_Schottky
Connections:
- net labels removed: VBAT_SW
- wire segments 113 -> 98
Changed lines of the file:
@@
 	1    0    0    -1
 $EndComp
-Wire Wire Line
-	9350 6250 9350 6300
-Text HLabel 9350 6300 3    50   Input ~ 0
-GND
-$Comp
-L Device:C C9
-U 1 1 609853E4
-P 9350 6100
-F 0 "C9" V 9098 6100 50  0000 C CNN
-F 1 "10 uF" V 9189 6100 50  0000 C CNN
-F 2 "Capacitor_SMD:C_1210_3225Metric" H 9388 5950 50  0001 C CNN
-F 3 "~" H 9350 6100 50  0001 C CNN
-F 4 "Taiyo Yuden" H 9350 6100 50  0001 C CNN "mfg1"
-F 5 "UMK325AB7106MMHP" H 9350 6100 50  0001 C CNN "mfg1pn"
-	1    9350 6100
-	1    0    0    1
-$EndComp
-Wire Wire Line
-	10150 6100 10150 6150
-Text HLabel 10150 6150 3    50   Input ~ 0
-GND
-Wire Wire Line
-	9700 5700 9750 5700
-Wire Wire Line
-	9400 5700 9350 5700
-Wire Wire Line
-	9350 5700 9350 5400
-Wire Wire Line
-	9350 5400 9700 5400
-Wire Wire Line
-	9350 5700 9350 5900
-Wire Wire Line
-	9350 5900 9750 5900
-Connection ~ 9350 5700
-Wire Wire Line
-	9350 5950 9350 5900
-Connection ~ 9350 5900
-Wire Wire Line
-	9700 5400 9700 5500
-Wire Wire Line
-	9700 5500 9750 5500
-$Comp
-L colinholzman:TPS61097A-33DBVR U3
-U 1 1 609EC946
-P 10150 5600
-F 0 "U3" H 10150 5967 50  0000 C CNN
-F 1 "TPS61097A-33DBVR" H 10150 5876 50  0000 C CNN
-F 2 "Package_TO_SOT_SMD:SOT-23-5" H 10150 4700 50  0001 C CNN
-F 3 "" H 10150 5450 50  0001 C CNN
-F 4 "Texas Instruments" H 10150 5600 50  0001 C CNN "mfg1"
-F 5 "TPS61097A-33DBVR" H 10150 5600 50  0001 C CNN "mfg1pn"
-	1    10150 5600
-	1    0    0    -1
-$EndComp
-Connection ~ 9350 5400
-Text HLabel 10650 5500 2    50   Input ~ 0
-+3V3
-Wire Wire Line
-	10600 5850 10600 5900
-Text HLabel 10600 5900 3    50   Input ~ 0
-GND
-$Comp
-L Device:C C10
-U 1 1 60994D70
-P 10600 5700
-F 0 "C10" H 10715 5654 50  0000 L CNN
-F 1 "10 uF" H 10715 5745 50  0000 L CNN
-F 2 "Capacitor_SMD:C_1210_3225Metric" H 10638 5550 50  0001 C CNN
-F 3 "~" H 10600 5700 50  0001 C CNN
-F 4 "Taiyo Yuden" H 10600 5700 50  0001 C CNN "mfg1"
-F 5 "UMK325AB7106MMHP" H 10600 5700 50  0001 C CNN "mfg1pn"
-	1    10600 5700
-	1    0    0    1
-$EndComp
-Wire Wire Line
-	10600 5550 10600 5500
-Wire Wire Line
-	10600 5500 10650 5500
-Wire Wire Line
-	10550 5500 10600 5500
-Connection ~ 10600 5500
-$Comp
-L Device:L L1
-U 1 1 60989E09
-P 9550 5700
-F 0 "L1" V 9350 5700 50  0000 C CNN
-F 1 "10 uH" V 9450 5700 50  0000 C CNN
-F 2 "colinholzman:DO3314-...MLC" H 9550 5700 50  0001 C CNN
-F 3 "~" H 9550 5700 50  0001 C CNN
-F 4 "Coilcraft" H 9550 5700 50  0001 C CNN "mfg1"
-F 5 "DO3314-103MLC" H 9550 5700 50  0001 C CNN "mfg1pn"
-	1    9550 5700
-	0    1    1    0
-$EndComp
-Wire Wire Line
-	9300 5400 9350 5400
 $Comp
 L Device:Battery BT1
@@
 Wire Wire Line
 	6800 5400 6750 5400
-Text HLabel 9300 5400 0    50   Input ~ 0
-VBAT_SW
 Text HLabel 7700 5400 0    50   Input ~ 0
 VBAT
 Wire Wire Line
 	7700 5400 7750 5400
-Text HLabel 8200 5500 2    50   Input ~ 0
-VBAT_SW
-Wire Wire Line
-	8200 5500 8150 5500
 $Comp
 L Switch:SW_SPDT SW1
@@
 Wire Wire Line
 	8550 2150 8500 2150
+$Comp
+L Device:D_Schottky D1
+U 1 1 60B4E39F
+P 8500 5500
+F 0 "D1" H 8500 5283 50  0000 C CNN
+F 1 "CUS08F30" H 8500 5374 50  0000 C CNN
+F 2 "Diode_SMD:D_SOD-323_HandSoldering" H 8500 5500 50  0001 C CNN
+F 3 "~" H 8500 5500 50  0001 C CNN
+F 4 "Toshiba" H 8500 5500 50  0001 C CNN "mfg1"
+F 5 "CUS08F30" H 8500 5500 50  0001 C CNN "mfg1pn"
+	1    8500 5500
+	-1   0    0    1
+$EndComp
+Wire Wire Line
+	8150 5500 8350 5500
+Wire Wire Line
+	8700 5500 8650 5500
+Text HLabel 8700 5500 2    50   Input ~ 0
++3V3
 $EndSCHEMATC

Commit message: Add A5135-H.
Parts:
- added U?: A5135-H, symbol colinholzman:A5135-H
Changed lines of the file:
@@
 Text HLabel 8700 5500 2    50   Input ~ 0
 +3V3
+$Comp
+L colinholzman:A5135-H U?
+U 1 1 60E16591
+P 10450 4100
+F 0 "U?" H 10450 4815 50  0000 C CNN
+F 1 "A5135-H" H 10450 4724 50  0000 C CNN
+F 2 "" H 10400 4000 50  0001 C CNN
+F 3 "" H 10400 4000 50  0001 C CNN
+	1    10450 4100
+	1    0    0    -1
+$EndComp
 $EndSCHEMATC

Commit message: Add L80 GPS, charge ic, and battery protection ic.
Parts:
- removed C6, C7: 0.1 uF, Capacitor_SMD:C_0805_2012Metric, symbol Device:C
- removed J3: Conn_01x03, Connector_JST:JST_PH_S3B-PH-K_1x03_P2.00mm_Horizontal, symbol Connector_Generic:Conn_01x03
- removed Q5: SI3443DDV-T1-GE3, Package_SO:TSOP-6_1.65x3.05mm_P0.95mm, symbol colinholzman:Si3443
- removed R8: 100k, Resistor_SMD:R_0805_2012Metric, symbol Device:R
- removed U2: LM3480-3.3, Package_TO_SOT_SMD:SOT-23, symbol Regulator_Linear:LM3480-3.3
- removed U?: A5135-H, symbol colinholzman:A5135-H
- added Q? (x2): CSD16301Q2, Package_SON:Texas_DQK, symbol Transistor_FET:CSD16301Q2
- added U3: L80-R, RF_GPS:Quectel_L80-R, symbol RF_GPS:L80-R
- added U?: MCP73831-2-OT, Package_TO_SOT_SMD:SOT-23-5, symbol Battery_Management:MCP73831-2-OT
- added U?: BQ297xy, Package_SON:WSON-6_1.5x1.5mm_P0.5mm, symbol Battery_Management:BQ297xy
- BT1: value Battery -> Lir2477; footprint cat-tracker-board:battery-board -> colinholzman:Keystone_3039
Connections:
- net labels removed: GPS_PWR
- wire segments 98 -> 77
Other:
- moved on the sheet: BT1, SW1

Commit message: Add charger support components.
Parts:
- removed U?: MCP73831-2-OT, Package_TO_SOT_SMD:SOT-23-5, symbol Battery_Management:MCP73831-2-OT
- added C? (x2): 4.7 uF, symbol Device:C
- added D?: SMAJ5.0A, Diode_SMD:D_SMA, symbol Diode:1.5KExxA
- added D?: LED, symbol Device:LED
- added R?: 14.7K, symbol Device:R
- added R?: 750, symbol Device:R
- added U?: MCP73831-2ACI/MC, symbol colinholzman:MCP7383*-*-MC
Connections:
- net labels added: VCELL
- wire segments 77 -> 102
Changed lines of the file:
@@
 Wire Wire Line
 	11250 1800 11300 1800
-Text HLabel 11250 1800 0    50   Input ~ 0
-USBDM
 $Comp
 L Power_Protection:PRTR5V0U2X D4
@@
 GND
 Text HLabel 5400 5100 2    50   Input ~ 0
-VBAT
+VCELL
 Wire Wire Line
 	5400 5100 5350 5100
@@
 $EndComp
 $Comp
-L Battery_Management:MCP73831-2-OT U?
-U 1 1 60E29AE2
-P 8050 1400
-F 0 "U?" H 8050 1881 50  0000 C CNN
-F 1 "MCP73831-2-OT" H 8050 1790 50  0000 C CNN
-F 2 "Package_TO_SOT_SMD:SOT-23-5" H 8100 1150 50  0001 L CIN
-F 3 "http://ww1.microchip.com/downloads/en/DeviceDoc/20001984g.pdf" H 7900 1350 50  0001 C CNN
-F 4 "Microchip" H 8050 1400 50  0001 C CNN "mfg1"
-F 5 "MCP73831T-2ATI/OT" H 8050 1400 50  0001 C CNN "mfg1pn"
-	1    8050 1400
-	1    0    0    -1
-$EndComp
-$Comp
 L Battery_Management:BQ297xy U?
 U 1 1 60E2FD2E
@@
 	1    0    0    -1
 $EndComp
+$Comp
+L colinholzman:MCP7383*-*-MC U?
+U 1 1 60E3AA2D
+P 8550 1550
+F 0 "U?" H 8550 1965 50  0000 C CNN
+F 1 "MCP73831-2ACI/MC" H 8550 1874 50  0000 C CNN
+F 2 "" H 8450 1450 50  0001 C CNN
+F 3 "" H 8450 1450 50  0001 C CNN
+F 4 "Microchip" H 8550 1550 50  0001 C CNN "mfg1"
+F 5 "MCP73831-2ACI/MC" H 8550 1550 50  0001 C CNN "mfg1pn"
+	1    8550 1550
+	1    0    0    -1
+$EndComp
+Wire Wire Line
+	8150 1600 8200 1600
+Wire Wire Line
+	8150 1700 8200 1700
+Wire Wire Line
+	8150 1400 8200 1400
+Wire Wire Line
+	8150 1500 8200 1500
+Text HLabel 11250 1800 0    50   Input ~ 0
+USBDM
+Wire Wire Line
+	8900 1600 8950 1600
+Text HLabel 8950 1600 2    50   Input ~ 0
+GND
+$Comp
+L Device:C C?
+U 1 1 60E4853F
+P 6800 1600
+F 0 "C?" H 6915 1646 50  0000 L CNN
+F 1 "4.7 uF" H 6915 1555 50  0000 L CNN
+F 2 "" H 6838 1450 50  0001 C CNN
+F 3 "~" H 6800 1600 50  0001 C CNN
+	1    6800 1600
+	1    0    0    -1
+$EndComp
+Wire Wire Line
+	6800 1350 6800 1400
+Text HLabel 6800 1350 1    50   Input ~ 0
+VUSB
+Wire Wire Line
+	6800 1750 6800 1800
+Text HLabel 6800 1800 3    50   Input ~ 0
+GND
+$Comp
+L Device:C C?
+U 1 1 60E4E50A
+P 8050 1900
+F 0 "C?" H 8165 1946 50  0000 L CNN
+F 1 "4.7 uF" H 8165 1855 50  0000 L CNN
+F 2 "" H 8088 1750 50  0001 C CNN
+F 3 "~" H 8050 1900 50  0001 C CNN
+	1    8050 1900
+	1    0    0    -1
+$EndComp
+Wire Wire Line
+	8050 2050 8050 2100
+Text HLabel 8050 2100 3    50   Input ~ 0
+GND
+$Comp
+L Device:R R?
+U 1 1 60E535B5
+P 9500 1650
+F 0 "R?" H 9570 1696 50  0000 L CNN
+F 1 "14.7K" H 9570 1605 50  0000 L CNN
+F 2 "" V 9430 1650 50  0001 C CNN
+F 3 "~" H 9500 1650 50  0001 C CNN
+	1    9500 1650
+	1    0    0    -1
+$EndComp
+Wire Wire Line
+	9500 1800 9500 1850
+Text HLabel 9500 1850 3    50   Input ~ 0
+GND
+Wire Wire Line
+	9500 1500 9500 1400
+Wire Wire Line
+	9500 1400 8900 1400
+Wire Wire Line
+	8150 1500 8150 1400
+Connection ~ 6800 1400
+Wire Wire Line
+	6800 1400 6800 1450
+Wire Wire Line
+	8150 1600 8150 1700
+Wire Wire Line
+	8050 1700 8150 1700
+Connection ~ 8050 1700
+Wire Wire Line
+	8050 1700 8050 1750
+Connection ~ 8150 1700
+Wire Wire Line
+	8000 1700 8050 1700
+Text HLabel 8000 1700 0    50   Input ~ 0
+VBAT
+$Comp
+L Diode:1.5KExxA D?
+U 1 1 60E8FB15
+P 7250 1600
+F 0 "D?" V 7204 1680 50  0000 L CNN
+F 1 "SMAJ5.0A" V 7295 1680 50  0000 L CNN
+F 2 "Diode_SMD:D_SMA" H 7250 1400 50  0001 C CNN
+F 3 "" H 7200 1600 50  0001 C CNN
+F 4 "Vishay" H 7250 1600 50  0001 C CNN "mfg1"
+F 5 "SMAJ5.0A-E3/61" H 7250 1600 50  0001 C CNN "mfg1pn"
+	1    7250 1600
+	0    1    1    0
+$EndComp
+Wire Wire Line
+	7250 1750 7250 1800
+Text HLabel 7250 1800 3    50   Input ~ 0
+GND
+Wire Wire Line
+	7250 1450 7250 1400
+Connection ~ 7250 1400
+Wire Wire Line
+	7250 1400 6800 1400
+Wire Wire Line
+	7250 1400 8150 1400
+Connection ~ 8150 1400
+$Comp
+L Device:R R?
+U 1 1 60EA1E99
+P 8950 2300
+F 0 "R?" H 9020 2346 50  0000 L CNN
+F 1 "750" H 9020 2255 50  0000 L CNN
+F 2 "" V 8880 2300 50  0001 C CNN
+F 3 "~" H 8950 2300 50  0001 C CNN
+	1    8950 2300
+	1    0    0    -1
+$EndComp
+$Comp
+L Device:LED D?
+U 1 1 60EA4C3A
+P 8950 1950
+F 0 "D?" V 8897 2030 50  0000 L CNN
+F 1 "LED" V 8988 2030 50  0000 L CNN
+F 2 "" H 8950 1950 50  0001 C CNN
+F 3 "~" H 8950 1950 50  0001 C CNN
+	1    8950 1950
+	0    1    1    0
+$EndComp
+Wire Wire Line
+	8950 1800 8950 1700
+Wire Wire Line
+	8950 1700 8900 1700
+Wire Wire Line
+	8950 2150 8950 2100
+Wire Wire Line
+	8950 2500 8950 2450
+Text HLabel 8950 2500 3    50   Input ~ 0
+VUSB
 $EndSCHEMATC

Commit message: Add support components for battery protection.
Parts:
- removed D1: CUS08F30, Diode_SMD:D_SOD-323_HandSoldering, symbol Device:D_Schottky
- added C?: 0.1 uF, symbol Device:C
- added R?: 2.2K, symbol Device:R
- added R?: 330, symbol Device:R
- U?: value BQ297xy -> BQ29737DSER
Connections:
- net labels removed: VCELL
- wire segments 102 -> 121
Other:
- moved on the sheet: BT1, Q?, SW1
Changed lines of the file:
@@
 L Device:Battery BT1
 U 1 1 6095446A
-P 5150 5100
-F 0 "BT1" V 4905 5100 50  0000 C CNN
-F 1 "Lir2477" V 4996 5100 50  0000 C CNN
-F 2 "colinholzman:Keystone_3039" V 5150 5160 50  0001 C CNN
-F 3 "~" V 5150 5160 50  0001 C CNN
-	1    5150 5100
-	0    1    1    0
-$EndComp
-Wire Wire Line
-	4950 5100 4900 5100
-Text HLabel 4900 5100 0    50   Input ~ 0
-GND
-Text HLabel 5400 5100 2    50   Input ~ 0
-VCELL
-Wire Wire Line
-	5400 5100 5350 5100
-Text HLabel 8650 5400 0    50   Input ~ 0
+P 7650 5350
+F 0 "BT1" H 7758 5396 50  0000 L CNN
+F 1 "Lir2477" H 7758 5305 50  0000 L CNN
+F 2 "colinholzman:Keystone_3039" V 7650 5410 50  0001 C CNN
+F 3 "~" V 7650 5410 50  0001 C CNN
+	1    7650 5350
+	1    0    0    -1
+$EndComp
+Text HLabel 7650 4600 1    50   Input ~ 0
 VBAT
-Wire Wire Line
-	8650 5400 8700 5400
+Text HLabel 9500 5550 0    50   Input ~ 0
+VBAT
+Wire Wire Line
+	9500 5550 9550 5550
 $Comp
 L Switch:SW_SPDT SW1
 U 1 1 60C01EB4
-P 8900 5400
-F 0 "SW1" H 8900 5685 50  0000 C CNN
-F 1 "PCM12SMTR" H 8900 5594 50  0000 C CNN
-F 2 "Button_Switch_SMD:SW_SPDT_PCM12" H 8900 5400 50  0001 C CNN
-F 3 "~" H 8900 5400 50  0001 C CNN
-F 4 "C&K" H 8900 5400 50  0001 C CNN "mfg1"
-F 5 "PCM12SMTR" H 8900 5400 50  0001 C CNN "mfg1pn"
-	1    8900 5400
-	1    0    0    -1
-$EndComp
-$Comp
-L Device:D_Schottky D1
-U 1 1 60B4E39F
-P 9450 5500
-F 0 "D1" H 9450 5283 50  0000 C CNN
-F 1 "CUS08F30" H 9450 5374 50  0000 C CNN
-F 2 "Diode_SMD:D_SOD-323_HandSoldering" H 9450 5500 50  0001 C CNN
-F 3 "~" H 9450 5500 50  0001 C CNN
-F 4 "Toshiba" H 9450 5500 50  0001 C CNN "mfg1"
-F 5 "CUS08F30" H 9450 5500 50  0001 C CNN "mfg1pn"
-	1    9450 5500
-	-1   0    0    1
-$EndComp
-Wire Wire Line
-	9100 5500 9300 5500
-Wire Wire Line
-	9650 5500 9600 5500
-Text HLabel 9650 5500 2    50   Input ~ 0
+P 9750 5550
+F 0 "SW1" H 9750 5835 50  0000 C CNN
+F 1 "PCM12SMTR" H 9750 5744 50  0000 C CNN
+F 2 "Button_Switch_SMD:SW_SPDT_PCM12" H 9750 5550 50  0001 C CNN
+F 3 "~" H 9750 5550 50  0001 C CNN
+F 4 "C&K" H 9750 5550 50  0001 C CNN "mfg1"
+F 5 "PCM12SMTR" H 9750 5550 50  0001 C CNN "mfg1pn"
+	1    9750 5550
+	1    0    0    -1
+$EndComp
+Text HLabel 10000 5650 2    50   Input ~ 0
 +3V3
 $Comp
@@
 P 6400 5200
 F 0 "U?" H 6400 5567 50  0000 C CNN
-F 1 "BQ297xy" H 6400 5476 50  0000 C CNN
+F 1 "BQ29737DSER" H 6400 5476 50  0000 C CNN
 F 2 "Package_SON:WSON-6_1.5x1.5mm_P0.5mm" H 6400 5550 50  0001 C CNN
 F 3 "http://www.ti.com/lit/ds/symlink/bq2970.pdf" H 6150 5400 50  0001 C CNN
@@
 F 6 "BQ29737DSET" H 6400 5200 50  0001 C CNN "mfg2pn"
 	1    6400 5200
-	1    0    0    -1
+	-1   0    0    -1
 $EndComp
 $Comp
 L Transistor_FET:CSD16301Q2 Q?
 U 1 1 60E3DE41
-P 7200 4850
-F 0 "Q?" H 7404 4896 50  0000 L CNN
-F 1 "CSD16301Q2" H 7404 4805 50  0000 L CNN
-F 2 "Package_SON:Texas_DQK" H 7400 4775 50  0001 L CIN
-F 3 "http://www.ti.com/lit/ds/symlink/csd16301q2.pdf" V 7200 4850 50  0001 L CNN
-	1    7200 4850
-	1    0    0    -1
+P 5950 5850
+F 0 "Q?" V 6199 5850 50  0000 C CNN
+F 1 "CSD16301Q2" V 6290 5850 50  0000 C CNN
+F 2 "Package_SON:Texas_DQK" H 6150 5775 50  0001 L CIN
+F 3 "http://www.ti.com/lit/ds/symlink/csd16301q2.pdf" V 5950 5850 50  0001 L CNN
+	1    5950 5850
+	0    -1   1    0
 $EndComp
 $Comp
 L Transistor_FET:CSD16301Q2 Q?
 U 1 1 60E42C5F
-P 7200 5500
-F 0 "Q?" H 7404 5546 50  0000 L CNN
-F 1 "CSD16301Q2" H 7404 5455 50  0000 L CNN
-F 2 "Package_SON:Texas_DQK" H 7400 5425 50  0001 L CIN
-F 3 "http://www.ti.com/lit/ds/symlink/csd16301q2.pdf" V 7200 5500 50  0001 L CNN
-	1    7200 5500
-	1    0    0    -1
+P 5400 5850
+F 0 "Q?" V 5649 5850 50  0000 C CNN
+F 1 "CSD16301Q2" V 5740 5850 50  0000 C CNN
+F 2 "Package_SON:Texas_DQK" H 5600 5775 50  0001 L CIN
+F 3 "http://www.ti.com/lit/ds/symlink/csd16301q2.pdf" V 5400 5850 50  0001 L CNN
+	1    5400 5850
+	0    1    1    0
 $EndComp
 $Comp
@@
 Text HLabel 8950 2500 3    50   Input ~ 0
 VUSB
+Wire Wire Line
+	5400 5650 5400 5100
+Wire Wire Line
+	5950 5650 5950 5300
+Wire Wire Line
+	5950 5300 6000 5300
+Wire Wire Line
+	5200 5950 5150 5950
+Text HLabel 5150 5950 0    50   Input ~ 0
+GND
+Wire Wire Line
+	6400 5500 6400 5950
+Wire Wire Line
+	6150 5950 6400 5950
+Wire Wire Line
+	6400 5950 7150 5950
+Wire Wire Line
+	7650 5550 7650 5950
+Connection ~ 6400 5950
+$Comp
+L Device:R R?
+U 1 1 60EE2DDD
+P 6850 5500
+F 0 "R?" H 6920 5546 50  0000 L CNN
+F 1 "2.2K" H 6920 5455 50  0000 L CNN
+F 2 "" V 6780 5500 50  0001 C CNN
+F 3 "~" H 6850 5500 50  0001 C CNN
+	1    6850 5500
+	1    0    0    -1
+$EndComp
+Wire Wire Line
+	6850 5350 6850 5300
+Wire Wire Line
+	6850 5300 6800 5300
+Wire Wire Line
+	6850 5700 6850 5650
+Text HLabel 6850 5700 3    50   Input ~ 0
+GND
+$Comp
+L Device:R R?
+U 1 1 60EEC27F
+P 7150 4900
+F 0 "R?" H 7220 4946 50  0000 L CNN
+F 1 "330" H 7220 4855 50  0000 L CNN
+F 2 "" V 7080 4900 50  0001 C CNN
+F 3 "~" H 7150 4900 50  0001 C CNN
+	1    7150 4900
+	1    0    0    -1
+$EndComp
+Wire Wire Line
+	7150 4750 7150 4700
+Wire Wire Line
+	7650 4700 7650 4600
+Wire Wire Line
+	7650 4700 7650 5150
+Connection ~ 7650 4700
+Wire Wire Line
+	6800 5100 7150 5100
+Wire Wire Line
+	7150 5100 7150 5050
+$Comp
+L Device:C C?
+U 1 1 60F00417
+P 7150 5350
+F 0 "C?" H 7265 5396 50  0000 L CNN
+F 1 "0.1 uF" H 7265 5305 50  0000 L CNN
+F 2 "" H 7188 5200 50  0001 C CNN
+F 3 "~" H 7150 5350 50  0001 C CNN
+	1    7150 5350
+	1    0    0    -1
+$EndComp
+Wire Wire Line
+	7150 5200 7150 5100
+Connection ~ 7150 5100
+Wire Wire Line
+	7150 5500 7150 5950
+Wire Wire Line
+	7150 4700 7650 4700
+Wire Wire Line
+	7150 5950 7650 5950
+Connection ~ 7150 5950
+Wire Wire Line
+	5600 5950 5750 5950
+Wire Wire Line
+	5400 5100 6000 5100
+Wire Wire Line
+	9950 5650 10000 5650
 $EndSCHEMATC

Commit message: Rescue symbols.
Parts:
- U1: symbol MCU_Microchip_SAMD:ATSAMD21E18A-A -> cat-tracker-board-rescue:ATSAMD21E18A-A-MCU_Microchip_SAMD
- U3: symbol RF_GPS:L80-R -> cat-tracker-board-rescue:L80-R-RF_GPS
Changed lines of the file:
@@
 nRESET
 $Comp
-L MCU_Microchip_SAMD:ATSAMD21E18A-A U1
+L cat-tracker-board-rescue:ATSAMD21E18A-A-MCU_Microchip_SAMD U1
 U 1 1 608CAFAA
 P 2350 4750
@@
 +3V3
 $Comp
-L RF_GPS:L80-R U3
+L cat-tracker-board-rescue:L80-R-RF_GPS U3
 U 1 1 60E2275D
 P 13600 7650

Commit message: Add MCP 1700 3.6V regulator.
Parts:
- added C? (x2): 1 uF, symbol Device:C
- added U?: MCP1700T-3602E/TT, Package_TO_SOT_SMD:SOT-23, symbol Regulator_Linear:MCP1700-3302E_SOT23
- J2: value USB_C_Receptacle_USB2.0 -> USB C
Connections:
- net +3V3: no longer C2.1, C3.2, FB1.1, R1.1, R2.1, SW1.3 (C), U1.30 (VDDIN), U4.13 (3.3V)
- net GND: now also C?.2, C?.2, U?.1 (GND)
- new net: C?.1, SW1.3 (C), U?.3 (VI)
- new net VDD: C2.1, C3.2, C?.1, FB1.1, R1.1, R2.1, U1.30 (VDDIN), U4.13 (3.3V), U?.2 (VO)
Other:
- note added: "Battery and protection"
- note added: "Charger"
- note added: "GPS"
- note added: "LoRa"
- note added: "USB C connector and protection"
- note added: "VDD regulator and power switch"
- moved on the sheet: BT1, C1, C2, C3, C4, C5, C?, D4, D?, FB1, J1, J2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
