File: main-board/cat-tracker-board.sch (KiCad schematic (older format))
At the start: 35 parts, among them J1 Conn_01x10, J2 USB C, J4 Conn_01x02, SW1 PCM12SMTR, U1 ATSAMD21E18A-A, U3 L80-R, U4 RFM95W-915S2

Commit message: Annotate, assign footprints, and assign part numbers.
Parts:
- removed J4: Conn_01x02, cat-tracker-board:RF-Solutions-CON-SMA-EDGE-S, symbol Connector_Generic:Conn_01x02
- BT1: mfg1 (none) -> Keystone; mfg1pn (none) -> 3039
- C1: mfg1 Samsung Electro-Mechanics -> Wurth Elektronik; mfg1pn CL21B105KBFNNNG -> 885012207051
- C10, C9: renamed from C?; footprint (none) -> Capacitor_SMD:C_0805_2012Metric; mfg1 (none) -> Wurth Elektronik; mfg1pn (none) -> 885012207051
- C2, C4: footprint Capacitor_SMD:C_1210_3225Metric -> Capacitor_SMD:C_0805_2012Metric; mfg1pn UMK325AB7106MMHP -> EMK212BB7106MG-T
- C6, C7: renamed from C?; footprint (none) -> Capacitor_SMD:C_0805_2012Metric; mfg1 (none) -> Murata Electronics; mfg1pn (none) -> GRM21BR71C475KE51L
- C8: renamed from C?; footprint (none) -> Capacitor_SMD:C_0805_2012Metric; mfg1 (none) -> AVX; mfg1pn (none) -> 08055C104KAT2A
- D2: renamed from D?; footprint (none) -> LED_SMD:LED_0805_2012Metric; mfg1 (none) -> Lite-On; mfg1pn (none) -> LTST-C171KRKT
- Q1, Q2: renamed from Q?; mfg1 (none) -> Texas Instruments; mfg1pn (none) -> CSD16301Q2
- R3: renamed from R?; footprint (none) -> Resistor_SMD:R_0805_2012Metric; mfg1 (none) -> Vishay / Dale; mfg1pn (none) -> CRCW08052K20FKEAC
- R4: renamed from R?; footprint (none) -> Resistor_SMD:R_0805_2012Metric; mfg1 (none) -> Vishay / Dale; mfg1pn (none) -> CRCW0805330RFKEAC
- R5: renamed from R?; footprint (none) -> Resistor_SMD:R_0805_2012Metric; mfg1 (none) -> Panasonic; mfg1pn (none) -> ERJ-6GEYJ751V
- R6: renamed from R?; value 14.7K -> 14K; footprint (none) -> Resistor_SMD:R_0805_2012Metric; mfg1 (none) -> Bourns; mfg1pn (none) -> CR0805-FX-1402ELF
- U5: renamed from U?; footprint (none) -> Package_DFN_QFN:DFN-8_2x2mm_P0.5mm
- gave numbers to parts that had none: 3
Changed lines of the file:
@@
 F 2 "Capacitor_SMD:C_0805_2012Metric" H 2088 4100 50  0001 C CNN
 F 3 "~" H 2050 4250 50  0001 C CNN
-F 4 "Samsung Electro-Mechanics" H 2050 4250 50  0001 C CNN "mfg1"
-F 5 "CL21B105KBFNNNG" H 2050 4250 50  0001 C CNN "mfg1pn"
+F 4 "Wurth Elektronik" H 2050 4250 50  0001 C CNN "mfg1"
+F 5 "885012207051" H 2050 4250 50  0001 C CNN "mfg1pn"
 	1    2050 4250
 	0    -1   1    0
@@
 F 0 "C2" V 1998 3350 50  0000 C CNN
 F 1 "10 uF" V 2089 3350 50  0000 C CNN
-F 2 "Capacitor_SMD:C_1210_3225Metric" H 2288 3200 50  0001 C CNN
+F 2 "Capacitor_SMD:C_0805_2012Metric" H 2288 3200 50  0001 C CNN
 F 3 "~" H 2250 3350 50  0001 C CNN
 F 4 "Taiyo Yuden" H 2250 3350 50  0001 C CNN "mfg1"
-F 5 "UMK325AB7106MMHP" H 2250 3350 50  0001 C CNN "mfg1pn"
+F 5 "EMK212BB7106MG-T" H 2250 3350 50  0001 C CNN "mfg1pn"
 	1    2250 3350
 	0    1    1    0
@@
 F 0 "C4" V 2798 3800 50  0000 C CNN
 F 1 "10 uF" V 2889 3800 50  0000 C CNN
-F 2 "Capacitor_SMD:C_1210_3225Metric" H 3088 3650 50  0001 C CNN
+F 2 "Capacitor_SMD:C_0805_2012Metric" H 3088 3650 50  0001 C CNN
 F 3 "~" H 3050 3800 50  0001 C CNN
 F 4 "Taiyo Yuden" H 3050 3800 50  0001 C CNN "mfg1"
-F 5 "UMK325AB7106MMHP" H 3050 3800 50  0001 C CNN "mfg1pn"
+F 5 "EMK212BB7106MG-T" H 3050 3800 50  0001 C CNN "mfg1pn"
 	1    3050 3800
 	0    -1   1    0
@@
 Text HLabel 1800 6400 0    50   Input ~ 0
 GPS_EN
-$Comp
-L Connector_Generic:Conn_01x02 J4
-U 1 1 608E9ABB
-P 14450 2000
-F 0 "J4" H 14530 1992 50  0000 L CNN
-F 1 "Conn_01x02" H 14530 1901 50  0000 L CNN
-F 2 "cat-tracker-board:RF-Solutions-CON-SMA-EDGE-S" H 14450 2000 50  0001 C CNN
-F 3 "~" H 14450 2000 50  0001 C CNN
-F 4 "RF Solutions" H 14450 2000 50  0001 C CNN "mfg1"
-F 5 "CON-SMA-EDGE-S" H 14450 2000 50  0001 C CNN "mfg1pn"
-	1    14450 2000
-	1    0    0    -1
-$EndComp
-Wire Wire Line
-	14250 2100 14200 2100
-Text HLabel 14200 2100 0    50   Input ~ 0
-GND
 Wire Wire Line
 	13700 2000 14250 2000
@@
 F 2 "colinholzman:Keystone_3039" V 8650 8160 50  0001 C CNN
 F 3 "~" V 8650 8160 50  0001 C CNN
+F 4 "Keystone" H 8650 8100 50  0001 C CNN "mfg1"
+F 5 "3039" H 8650 8100 50  0001 C CNN "mfg1pn"
 	1    8650 8100
 	1    0    0    -1
@@
 $EndComp
 $Comp
-L Battery_Management:BQ297xy U?
+L Battery_Management:BQ297xy U2
 U 1 1 60E2FD2E
 P 7400 7950
-F 0 "U?" H 7400 8317 50  0000 C CNN
+F 0 "U2" H 7400 8317 50  0000 C CNN
 F 1 "BQ29737DSER" H 7400 8226 50  0000 C CNN
 F 2 "Package_SON:WSON-6_1.5x1.5mm_P0.5mm" H 7400 8300 50  0001 C CNN
@@
 $EndComp
 $Comp
-L Transistor_FET:CSD16301Q2 Q?
+L Transistor_FET:CSD16301Q2 Q2
 U 1 1 60E3DE41
 P 6950 8600
-F 0 "Q?" V 7199 8600 50  0000 C CNN
+F 0 "Q2" V 7199 8600 50  0000 C CNN
 F 1 "CSD16301Q2" V 7290 8600 50  0000 C CNN
 F 2 "Package_SON:Texas_DQK" H 7150 8525 50  0001 L CIN
 F 3 "http://www.ti.com/lit/ds/symlink/csd16301q2.pdf" V 6950 8600 50  0001 L CNN
+F 4 "Texas Instruments" H 6950 8600 50  0001 C CNN "mfg1"
+F 5 "CSD16301Q2" H 6950 8600 50  0001 C CNN "mfg1pn"
 	1    6950 8600
 	0    -1   1    0
 $EndComp
 $Comp
-L Transistor_FET:CSD16301Q2 Q?
+L Transistor_FET:CSD16301Q2 Q1
 U 1 1 60E42C5F
 P 6400 8600
-F 0 "Q?" V 6649 8600 50  0000 C CNN
+F 0 "Q1" V 6649 8600 50  0000 C CNN
 F 1 "CSD16301Q2" V 6740 8600 50  0000 C CNN
 F 2 "Package_SON:Texas_DQK" H 6600 8525 50  0001 L CIN
 F 3 "http://www.ti.com/lit/ds/symlink/csd16301q2.pdf" V 6400 8600 50  0001 L CNN
+F 4 "Texas Instruments" H 6400 8600 50  0001 C CNN "mfg1"
+F 5 "CSD16301Q2" H 6400 8600 50  0001 C CNN "mfg1pn"
 	1    6400 8600
 	0    1    1    0
 $EndComp
 $Comp
-L colinholzman:MCP7383*-*-MC U?
+L colinholzman:MCP7383*-*-MC U5
 U 1 1 60E3AA2D
 P 7850 5000
-F 0 "U?" H 7850 5415 50  0000 C CNN
+F 0 "U5" H 7850 5415 50  0000 C CNN
 F 1 "MCP73831-2ACI/MC" H 7850 5324 50  0000 C CNN
-F 2 "" H 7750 4900 50  0001 C CNN
+F 2 "Package_DFN_QFN:DFN-8_2x2mm_P0.5mm" H 7750 4900 50  0001 C CNN
 F 3 "" H 7750 4900 50  0001 C CNN
 F 4 "Microchip" H 7850 5000 50  0001 C CNN "mfg1"
@@
 GND
 $Comp
-L Device:C C?
+L Device:C C6
 U 1 1 60E4853F
 P 6100 5050
-F 0 "C?" H 6215 5096 50  0000 L CNN
+F 0 "C6" H 6215 5096 50  0000 L CNN
 F 1 "4.7 uF" H 6215 5005 50  0000 L CNN
-F 2 "" H 6138 4900 50  0001 C CNN
+F 2 "Capacitor_SMD:C_0805_2012Metric" H 6138 4900 50  0001 C CNN
 F 3 "~" H 6100 5050 50  0001 C CNN
+F 4 "Murata Electronics" H 6100 5050 50  0001 C CNN "mfg1"
+F 5 "GRM21BR71C475KE51L" H 6100 5050 50  0001 C CNN "mfg1pn"
 	1    6100 5050
 	1    0    0    -1
@@
 GND
 $Comp
-L Device:C C?
+L Device:C C7
 U 1 1 60E4E50A
 P 7350 5350
-F 0 "C?" H 7465 5396 50  0000 L CNN
+F 0 "C7" H 7465 5396 50  0000 L CNN
 F 1 "4.7 uF" H 7465 5305 50  0000 L CNN
-F 2 "" H 7388 5200 50  0001 C CNN
+F 2 "Capacitor_SMD:C_0805_2012Metric" H 7388 5200 50  0001 C CNN
 F 3 "~" H 7350 5350 50  0001 C CNN
+F 4 "Murata Electronics" H 7350 5350 50  0001 C CNN "mfg1"
+F 5 "GRM21BR71C475KE51L" H 7350 5350 50  0001 C CNN "mfg1pn"
 	1    7350 5350
 	1    0    0    -1
@@
 GND
 $Comp
-L Device:R R?
+L Device:R R6
 U 1 1 60E535B5
 P 8800 5100
-F 0 "R?" H 8870 5146 50  0000 L CNN
-F 1 "14.7K" H 8870 5055 50  0000 L CNN
-F 2 "" V 8730 5100 50  0001 C CNN
+F 0 "R6" H 8870 5146 50  0000 L CNN
+F 1 "14K" H 8870 5055 50  0000 L CNN
+F 2 "Resistor_SMD:R_0805_2012Metric" V 8730 5100 50  0001 C CNN
 F 3 "~" H 8800 5100 50  0001 C CNN
+F 4 "Bourns" H 8800 5100 50  0001 C CNN "mfg1"
+F 5 "CR0805-FX-1402ELF" H 8800 5100 50  0001 C CNN "mfg1pn"
 	1    8800 5100
 	1    0    0    -1
@@
 VBAT
 $Comp
-L Diode:1.5KExxA D?
+L Diode:1.5KExxA D1
 U 1 1 60E8FB15
 P 6550 5050
-F 0 "D?" V 6504 5130 50  0000 L CNN
+F 0 "D1" V 6504 5130 50  0000 L CNN
 F 1 "SMAJ5.0A" V 6595 5130 50  0000 L CNN
 F 2 "Diode_SMD:D_SMA" H 6550 4850 50  0001 C CNN
@@
 Connection ~ 7450 4850
 $Comp
-L Device:R R?
+L Device:R R5
 U 1 1 60EA1E99
 P 8250 5750
-F 0 "R?" H 8320 5796 50  0000 L CNN
+F 0 "R5" H 8320 5796 50  0000 L CNN
 F 1 "750" H 8320 5705 50  0000 L CNN
-F 2 "" V 8180 5750 50  0001 C CNN
+F 2 "Resistor_SMD:R_0805_2012Metric" V 8180 5750 50  0001 C CNN
 F 3 "~" H 8250 5750 50  0001 C CNN
+F 4 "Panasonic" H 8250 5750 50  0001 C CNN "mfg1"
+F 5 "ERJ-6GEYJ751V" H 8250 5750 50  0001 C CNN "mfg1pn"
 	1    8250 5750
 	1    0    0    -1
 $EndComp
 $Comp
-L Device:LED D?
+L Device:LED D2
 U 1 1 60EA4C3A
 P 8250 5400
-F 0 "D?" V 8197 5480 50  0000 L CNN
+F 0 "D2" V 8197 5480 50  0000 L CNN
 F 1 "LED" V 8288 5480 50  0000 L CNN
-F 2 "" H 8250 5400 50  0001 C CNN
+F 2 "LED_SMD:LED_0805_2012Metric" H 8250 5400 50  0001 C CNN
 F 3 "~" H 8250 5400 50  0001 C CNN
+F 4 "Lite-On" H 8250 5400 50  0001 C CNN "mfg1"
+F 5 "LTST-C171KRKT" H 8250 5400 50  0001 C CNN "mfg1pn"
 	1    8250 5400
 	0    1    1    0
@@
 Connection ~ 7400 8700
 $Comp
-L Device:R R?
+L Device:R R3
 U 1 1 60EE2DDD
 P 7850 8250
-F 0 "R?" H 7920 8296 50  0000 L CNN
+F 0 "R3" H 7920 8296 50  0000 L CNN
 F 1 "2.2K" H 7920 8205 50  0000 L CNN
-F 2 "" V 7780 8250 50  0001 C CNN
+F 2 "Resistor_SMD:R_0805_2012Metric" V 7780 8250 50  0001 C CNN
 F 3 "~" H 7850 8250 50  0001 C CNN
+F 4 "Vishay / Dale" H 7850 8250 50  0001 C CNN "mfg1"
+F 5 "CRCW08052K20FKEAC" H 7850 8250 50  0001 C CNN "mfg1pn"
 	1    7850 8250
 	1    0    0    -1
@@
 GND
 $Comp
-L Device:R R?
+L Device:R R4
 U 1 1 60EEC27F
 P 8150 7650
-F 0 "R?" H 8220 7696 50  0000 L CNN
+F 0 "R4" H 8220 7696 50  0000 L CNN
 F 1 "330" H 8220 7605 50  0000 L CNN
-F 2 "" V 8080 7650 50  0001 C CNN
+F 2 "Resistor_SMD:R_0805_2012Metric" V 8080 7650 50  0001 C CNN
 F 3 "~" H 8150 7650 50  0001 C CNN
+F 4 "Vishay / Dale" H 8150 7650 50  0001 C CNN "mfg1"
+F 5 "CRCW0805330RFKEAC" H 8150 7650 50  0001 C CNN "mfg1pn"
 	1    8150 7650
 	1    0    0    -1
@@
 	8150 7850 8150 7800
 $Comp
-L Device:C C?
+L Device:C C8
 U 1 1 60F00417
 P 8150 8100
-F 0 "C?" H 8265 8146 50  0000 L CNN
+F 0 "C8" H 8265 8146 50  0000 L CNN
 F 1 "0.1 uF" H 8265 8055 50  0000 L CNN
-F 2 "" H 8188 7950 50  0001 C CNN
+F 2 "Capacitor_SMD:C_0805_2012Metric" H 8188 7950 50  0001 C CNN
 F 3 "~" H 8150 8100 50  0001 C CNN
+F 4 "AVX" H 8150 8100 50  0001 C CNN "mfg1"
+F 5 "08055C104KAT2A" H 8150 8100 50  0001 C CNN "mfg1pn"
 	1    8150 8100
 	1    0    0    -1
@@
 	11600 8050 11650 8050
 $Comp
-L Regulator_Linear:MCP1700-3302E_SOT23 U?
+L Regulator_Linear:MCP1700-3302E_SOT23 U6
 U 1 1 60E5E54D
 P 11300 8050
-F 0 "U?" H 11300 8292 50  0000 C CNN
+F 0 "U6" H 11300 8292 50  0000 C CNN
 F 1 "MCP1700T-3602E/TT" H 11300 8201 50  0000 C CNN
 F 2 "Package_TO_SOT_SMD:SOT-23" H 11300 8275 50  0001 C CNN
@@
 	2450 3300 2450 3350
 $Comp
-L Device:C C?
+L Device:C C9
 U 1 1 60E98BA9
 P 10800 8250
-F 0 "C?" H 10915 8296 50  0000 L CNN
+F 0 "C9" H 10915 8296 50  0000 L CNN
 F 1 "1 uF" H 10915 8205 50  0000 L CNN
-F 2 "" H 10838 8100 50  0001 C CNN
+F 2 "Capacitor_SMD:C_0805_2012Metric" H 10838 8100 50  0001 C CNN
 F 3 "~" H 10800 8250 50  0001 C CNN
+F 4 "Wurth Elektronik" H 10800 8250 50  0001 C CNN "mfg1"
+F 5 "885012207051" H 10800 8250 50  0001 C CNN "mfg1pn"
 	1    10800 8250
 	1    0    0    -1
@@
 GND
 $Comp
-L Device:C C?
+L Device:C C10
 U 1 1 60EA6B30
 P 11650 8250
-F 0 "C?" H 11765 8296 50  0000 L CNN
+F 0 "C10" H 11765 8296 50  0000 L CNN
 F 1 "1 uF" H 11765 8205 50  0000 L CNN
-F 2 "" H 11688 8100 50  0001 C CNN
+F 2 "Capacitor_SMD:C_0805_2012Metric" H 11688 8100 50  0001 C CNN
 F 3 "~" H 11650 8250 50  0001 C CNN
+F 4 "Wurth Elektronik" H 11650 8250 50  0001 C CNN "mfg1"
+F 5 "885012207051" H 11650 8250 50  0001 C CNN "mfg1pn"
 	1    11650 8250
 	1    0    0    -1
